File: tomu.sch (KiCad schematic (older format))
At the start: 15 parts, among them P1 USART0, P2 DEBUG, P3 USB-PCB, U1 EFM32HG309

Commit message: wip commit: half-done rework
The big difference with v0.4 is a large cutout on the side to facilitate
mating with an enclosure.  This necessitates many changes to the board
layout.

Signed-off-by: Sean Cross <sean@xobs.io>
Parts:
- removed P1: USART0, Pin_Headers:Pin_Header_Angled_1x04, symbol CONN_01X04
- removed P2: DEBUG, Pin_Headers:Pin_Header_Angled_1x04, symbol CONN_01X04
- added P1: TEST, symbol CONN_01X03
- added P2: DEBUG, usb-pcb:SMT-5pin, symbol CONN_01X05
- D1, D2: symbol LED -> LED-RESCUE-tomu
- W1, W2: symbol TEST -> TEST-RESCUE-tomu
Connections:
- net labels added: +3.3V, +5V, RESET/
- net labels removed: LEU0_RX, LEU0_TX
- wire segments 78 -> 94
- no-connect marks 3 -> 4
Other:
- moved on the sheet: C3, P3
